Commit message: namespace=base works

File: husky_gazebo/urdf/description.gazebo.xacro (robot description, xacro)
@@ -25,6 +25,6 @@
   <xacro:arg name="ur5_enabled" default="false" />
   <xacro:arg name="kinect_enabled" default="false" />
-  <xacro:arg name="namespace_with_slash" default="/base" />
-  <xacro:arg name="prefix_without_underscore" default="base" />
+  <xacro:arg name="namespace_with_slash" default="/" />
+  <xacro:arg name="prefix_with_underscore" default="" />
   <xacro:include filename="$(find husky_description)/urdf/husky.urdf.xacro" />
   <xacro:include filename="$(find husky_gazebo)/urdf/husky.gazebo.xacro" />
@@ -35,5 +35,5 @@
     </plugin>
   </gazebo>
-  <xacro:husky_robot />
-  <xacro:husky_robot_gazebo namespace_with_slash="$(arg namespace_with_slash)" />
+  <xacro:husky_robot extra_prefix="$(arg prefix_with_underscore)" />
+  <xacro:husky_robot_gazebo namespace_with_slash="$(arg namespace_with_slash)" extra_prefix="$(arg prefix_with_underscore)" />
 </robot>

File: husky_gazebo/urdf/husky.gazebo.xacro (robot description, xacro)
@@ -23,10 +23,10 @@
 <robot name="husky_robot_gazebo" xmlns:xacro="http://ros.org/wiki/xacro">
   <xacro:include filename="$(find husky_gazebo)/urdf/accessories/kinect_camera.gazebo.xacro"/>
-  <xacro:macro name="husky_robot_gazebo" params="namespace_with_slash">
+  <xacro:macro name="husky_robot_gazebo" params="namespace_with_slash extra_prefix">
     <gazebo>
       <plugin name="imu_controller" filename="libhector_gazebo_ros_imu.so">
         <robotNamespace>$(arg namespace_with_slash)</robotNamespace>
         <updateRate>50.0</updateRate>
-        <bodyName>base_link</bodyName>
+        <bodyName>${extra_prefix}base_link</bodyName>
         <topicName>imu/data</topicName>
         <accelDrift>0.005 0.005 0.005</accelDrift>
@@ -43,6 +43,6 @@
         <updateRate>40</updateRate>
         <robotNamespace>/</robotNamespace>
-        <bodyName>base_link</bodyName>
-        <frameId>base_link</frameId>
+        <bodyName>${extra_prefix}base_link</bodyName>
+        <frameId>${extra_prefix}base_link</frameId>
         <topicName>navsat/fix</topicName>
         <velocityTopicName>navsat/vel</velocityTopicName>
@@ -56,28 +56,28 @@
     <xacro:if value="$(arg ur5_enabled)">
       <!--Remove when https://github.com/ros-industrial/universal_robot/pull/168 is resolved -->
-      <gazebo reference="ur5_arm_shoulder_link">
+      <gazebo reference="${extra_prefix}ur5_arm_shoulder_link">
         <selfCollide>true</selfCollide>
       </gazebo>
-      <gazebo reference="ur5_arm_upper_arm_link">
+      <gazebo reference="${extra_prefix}ur5_arm_upper_arm_link">
         <selfCollide>true</selfCollide>
       </gazebo>
-      <gazebo reference="ur5_arm_forearm_link">
+      <gazebo reference="${extra_prefix}ur5_arm_forearm_link">
         <selfCollide>true</selfCollide>
       </gazebo>
-      <gazebo reference="ur5_arm_wrist_1_link">
+      <gazebo reference="${extra_prefix}ur5_arm_wrist_1_link">
         <selfCollide>true</selfCollide>
       </gazebo>
-      <gazebo reference="ur5_arm_wrist_3_link">
+      <gazebo reference="${extra_prefix}ur5_arm_wrist_3_link">
        <selfCollide>true</selfCollide>
       </gazebo>
-      <gazebo reference="ur5_arm_wrist_2_link">
+      <gazebo reference="${extra_prefix}ur5_arm_wrist_2_link">
         <selfCollide>true</selfCollide>
       </gazebo>
-      <gazebo reference="ur5_arm_ee_link">
+      <gazebo reference="${extra_prefix}ur5_arm_ee_link">
         <selfCollide>true</selfCollide>
       </gazebo>
     </xacro:if>
     <xacro:if value="$(arg kinect_enabled)">
-      <xacro:kinect_camera_gazebo prefix="camera" namespace_with_slash="$(arg namespace_with_slash)" />
+      <xacro:kinect_camera_gazebo prefix="${extra_prefix}camera" namespace_with_slash="$(arg namespace_with_slash)" />
     </xacro:if>
   </xacro:macro>
