Commit message: gazebo with namespace working

File: husky_gazebo/urdf/accessories/kinect_camera.gazebo.xacro (robot description, xacro)
@@ -1,5 +1,5 @@
 <?xml version="1.0"?>
 <root xmlns:xacro="http://ros.org/wiki/xacro">
-<xacro:macro name="kinect_camera_gazebo" params="prefix">
+<xacro:macro name="kinect_camera_gazebo" params="prefix namespace_with_slash">
   <joint name="${prefix}_optical_joint" type="fixed">
     <origin xyz="0 0 0" rpy="-1.5708 0 -1.5708"/>
@@ -25,4 +25,5 @@
       </camera>
       <plugin name="kinect_${prefix}_controller" filename="libgazebo_ros_openni_kinect.so">
+        <robotNamespace>$(arg namespace_with_slash)</robotNamespace>
         <cameraName>${prefix}</cameraName>
         <alwaysOn>true</alwaysOn>

File: husky_gazebo/urdf/description.gazebo.xacro (robot description, xacro)
@@ -25,4 +25,6 @@
   <xacro:arg name="ur5_enabled" default="false" />
   <xacro:arg name="kinect_enabled" default="false" />
+  <xacro:arg name="namespace_with_slash" default="/base" />
+  <xacro:arg name="prefix_without_underscore" default="base" />
   <xacro:include filename="$(find husky_description)/urdf/husky.urdf.xacro" />
   <xacro:include filename="$(find husky_gazebo)/urdf/husky.gazebo.xacro" />
@@ -30,8 +32,8 @@
   <gazebo>
     <plugin name="gazebo_ros_control" filename="libgazebo_ros_control.so">
-      <robotNamespace>/xxxxx</robotNamespace>
+      <robotNamespace>$(arg namespace_with_slash)</robotNamespace>
     </plugin>
   </gazebo>
   <xacro:husky_robot />
-  <xacro:husky_robot_gazebo />
+  <xacro:husky_robot_gazebo namespace_with_slash="$(arg namespace_with_slash)" />
 </robot>

File: husky_gazebo/urdf/husky.gazebo.xacro (robot description, xacro)
@@ -23,8 +23,8 @@
 <robot name="husky_robot_gazebo" xmlns:xacro="http://ros.org/wiki/xacro">
   <xacro:include filename="$(find husky_gazebo)/urdf/accessories/kinect_camera.gazebo.xacro"/>
-  <xacro:macro name="husky_robot_gazebo">
+  <xacro:macro name="husky_robot_gazebo" params="namespace_with_slash">
     <gazebo>
       <plugin name="imu_controller" filename="libhector_gazebo_ros_imu.so">
-        <robotNamespace>/xxxxx</robotNamespace>
+        <robotNamespace>$(arg namespace_with_slash)</robotNamespace>
         <updateRate>50.0</updateRate>
         <bodyName>base_link</bodyName>
@@ -40,5 +40,5 @@
     <gazebo>
       <plugin name="gps_controller" filename="libhector_gazebo_ros_gps.so">
-        <robotNamespace>/xxxxx</robotNamespace>
+        <robotNamespace>$(arg namespace_with_slash)</robotNamespace>
         <updateRate>40</updateRate>
         <robotNamespace>/</robotNamespace>
@@ -79,5 +79,5 @@
     </xacro:if>
     <xacro:if value="$(arg kinect_enabled)">
-      <xacro:kinect_camera_gazebo prefix="camera"/>
+      <xacro:kinect_camera_gazebo prefix="camera" namespace_with_slash="$(arg namespace_with_slash)" />
     </xacro:if>
   </xacro:macro>

Commit message: make param vs arg tidy

File: husky_gazebo/urdf/accessories/kinect_camera.gazebo.xacro (robot description, xacro)
@@ -25,5 +25,5 @@
       </camera>
       <plugin name="kinect_${prefix}_controller" filename="libgazebo_ros_openni_kinect.so">
-        <robotNamespace>$(arg namespace_with_slash)</robotNamespace>
+        <robotNamespace>${namespace_with_slash}</robotNamespace>
         <cameraName>${prefix}</cameraName>
         <alwaysOn>true</alwaysOn>

File: husky_gazebo/urdf/description.gazebo.xacro (robot description, xacro)
@@ -22,9 +22,9 @@
 -->
 <robot name="husky_robot_gazebo" xmlns:xacro="http://ros.org/wiki/xacro">
-  <xacro:arg name="laser_enabled" default="true" />
-  <xacro:arg name="ur5_enabled" default="false" />
-  <xacro:arg name="kinect_enabled" default="false" />
-  <xacro:arg name="namespace_with_slash" default="/" />
-  <xacro:arg name="prefix_with_underscore" default="" />
+  <xacro:arg name="laser_enabled" default="??laser_enabled??" />
+  <xacro:arg name="ur5_enabled" default="??ur5_enabled??" />
+  <xacro:arg name="kinect_enabled" default="??kinect_enabled??" />
+  <xacro:arg name="namespace_with_slash" default="??namespace_with_slash??" />
+  <xacro:arg name="prefix_with_underscore" default="??prefix_with_underscore??" />
   <xacro:include filename="$(find husky_description)/urdf/husky.urdf.xacro" />
   <xacro:include filename="$(find husky_gazebo)/urdf/husky.gazebo.xacro" />
@@ -35,5 +35,15 @@
     </plugin>
   </gazebo>
-  <xacro:husky_robot extra_prefix="$(arg prefix_with_underscore)" />
-  <xacro:husky_robot_gazebo namespace_with_slash="$(arg namespace_with_slash)" extra_prefix="$(arg prefix_with_underscore)" />
+  <xacro:husky_robot
+    extra_prefix="$(arg prefix_with_underscore)"
+    laser_enabled="$(arg laser_enabled)"
+    ur5_enabled="$(arg ur5_enabled)"
+    kinect_enabled="$(arg kinect_enabled)"
+    />
+  <xacro:husky_robot_gazebo
+    namespace_with_slash="$(arg namespace_with_slash)"
+    extra_prefix="$(arg prefix_with_underscore)"
+    ur5_enabled="$(arg ur5_enabled)"
+    kinect_enabled="$(arg kinect_enabled)"
+    />
 </robot>

File: husky_gazebo/urdf/husky.gazebo.xacro (robot description, xacro)
@@ -23,8 +23,9 @@
 <robot name="husky_robot_gazebo" xmlns:xacro="http://ros.org/wiki/xacro">
   <xacro:include filename="$(find husky_gazebo)/urdf/accessories/kinect_camera.gazebo.xacro"/>
-  <xacro:macro name="husky_robot_gazebo" params="namespace_with_slash extra_prefix">
+  <xacro:macro name="husky_robot_gazebo"
+    params="namespace_with_slash extra_prefix ur5_enabled kinect_enabled">
     <gazebo>
       <plugin name="imu_controller" filename="libhector_gazebo_ros_imu.so">
-        <robotNamespace>$(arg namespace_with_slash)</robotNamespace>
+        <robotNamespace>${namespace_with_slash}</robotNamespace>
         <updateRate>50.0</updateRate>
         <bodyName>${extra_prefix}base_link</bodyName>
@@ -40,5 +41,5 @@
     <gazebo>
       <plugin name="gps_controller" filename="libhector_gazebo_ros_gps.so">
-        <robotNamespace>$(arg namespace_with_slash)</robotNamespace>
+        <robotNamespace>${namespace_with_slash}</robotNamespace>
         <updateRate>40</updateRate>
         <robotNamespace>/</robotNamespace>
@@ -54,5 +55,5 @@
       </plugin>
     </gazebo>
-    <xacro:if value="$(arg ur5_enabled)">
+    <xacro:if value="${ur5_enabled}">
       <!--Remove when https://github.com/ros-industrial/universal_robot/pull/168 is resolved -->
       <gazebo reference="${extra_prefix}ur5_arm_shoulder_link">
@@ -78,6 +79,6 @@
       </gazebo>
     </xacro:if>
-    <xacro:if value="$(arg kinect_enabled)">
-      <xacro:kinect_camera_gazebo prefix="${extra_prefix}camera" namespace_with_slash="$(arg namespace_with_slash)" />
+    <xacro:if value="${kinect_enabled}">
+      <xacro:kinect_camera_gazebo prefix="${extra_prefix}camera" namespace_with_slash="${namespace_with_slash}" />
     </xacro:if>
   </xacro:macro>
